File: Hardware/esp32-V2.kicad_pcb (KiCad board)
At the start: 4 copper layers, 103.7 x 68 mm, 87 parts, among them J1 Conn_01x01_Socket, J10 MSD-4-A, J2 Conn_01x01_Socket, J3 Conn_01x08, J4 USB_C_Receptacle_USB2.0_16P, J5 PM254-1-17-Z-8.5, J6 ER-CON06HT-1, J7 Conn_01x01_Socket, J8 Conn_01x01_Socket, J9 ER-CON50HT-1, Q1 DMP3015LSS-13, Q2 MMBT3904, Q3 MMBT3904, SW1 SW_Push, SW2 SW_Push, SW3 SW_Push_DPDT, U2 TPS61170DRVR, U3 TPS61022, U4 ESP32-S31-WROOM-3-N16R16V, U5 LT1963AEST-3.3#TRPBF, U6 CN3158, U7 TPS63700

Commit message: Schematic Done
Parts:
- removed the C1 at (206.8, 48.7)
- removed the C14 at (196.9, 36.1)
- removed the C26 at (136.1, 93.8)
- removed JP1, JP3: SolderJumper_2_Bridged, Jumper:SolderJumper-2_P1.3mm_Bridged_Pad1.0x1.5mm
- removed JP2: SolderJumper_2_Open, Jumper:SolderJumper-2_P1.3mm_Open_TrianglePad1.0x1.5mm
- removed the Q2 at (198.0, 28.5)
- removed Q3: MMBT3904, Package_TO_SOT_SMD:SOT-23
- removed R15: 10k, Resistor_SMD:R_0402_1005Metric
- removed REF**: KiCad-Logo2_12mm_SilkScreen, Symbol:KiCad-Logo2_12mm_SilkScreen
- added C28: 10uF, Capacitor_SMD:C_0402_1005Metric, F.Cu at (213.5, 48.2)
- added C29: 10uF, Capacitor_SMD:C_0402_1005Metric, F.Cu at (212.2, 78.5)
- added C30: 4.7uF, Capacitor_SMD:C_0402_1005Metric, F.Cu at (165.2, 83.2)
- added C31: 1nF, Capacitor_SMD:C_0402_1005Metric, F.Cu at (169.0, 110.2)
- added C32: 1nF, Capacitor_SMD:C_0402_1005Metric, F.Cu at (181.3, 110.2)
- added C33: 4.7uF, Capacitor_SMD:C_0402_1005Metric, F.Cu at (165.2, 85.2)
- added C34: 4.7uF, Capacitor_SMD:C_0402_1005Metric, F.Cu at (165.2, 87.1)
- added C35: 4.7uF, Capacitor_SMD:C_0402_1005Metric, F.Cu at (165.2, 89.1)
- added C7: 470nF, Capacitor_SMD:C_0402_1005Metric, F.Cu at (93.2, 78.2)
- added C8: 470nF, Capacitor_SMD:C_0402_1005Metric, F.Cu at (93.2, 80.2)
- added C9: 10uF, Capacitor_SMD:C_0402_1005Metric, F.Cu at (165.2, 81.2)
- added D10: BSDFN2C031U, PCM_JLCPCB:D_DFN1006-2L, F.Cu at (189.8, 42.6)
- added D11: BSDFN2C031U, PCM_JLCPCB:D_DFN1006-2L, F.Cu at (189.8, 44.3)
- added D12: BSDFN2C031U, PCM_JLCPCB:D_DFN1006-2L, F.Cu at (189.8, 46.0)
- added D13: BSDFN2C031U, PCM_JLCPCB:D_DFN1006-2L, F.Cu at (229.3, 110.8)
- added D14: BSDFN2C031U, PCM_JLCPCB:D_DFN1006-2L, F.Cu at (229.3, 112.5)
- added D15: D_Schottky, Diode_SMD:D_SOD-123F, F.Cu at (94.5, 91.4)
- added D2: BSDFN2C031U, PCM_JLCPCB:D_DFN1006-2L, F.Cu at (189.8, 36.0)
- added D4: BSDFN2C031U, PCM_JLCPCB:D_DFN1006-2L, F.Cu at (189.8, 37.7)
- added D5: BSDFN2C031U, PCM_JLCPCB:D_DFN1006-2L, F.Cu at (189.8, 39.4)
- added D9: BSDFN2C031U, PCM_JLCPCB:D_DFN1006-2L, F.Cu at (189.8, 41.0)
- added F1: BSMD1812-300-16V, Fuse:Fuse_1812_4532Metric_Pad1.30x3.40mm_HandSolder, F.Cu at (136.2, 67.2)
- added F2: BSMD1812-300-16V, Fuse:Fuse_1812_4532Metric_Pad1.30x3.40mm_HandSolder, F.Cu at (131.5, 67.2)
- added F3: BSMD1812-300-16V, Fuse:Fuse_1812_4532Metric_Pad1.30x3.40mm_HandSolder, F.Cu at (210.2, 103.2)
- added L9: 10uH, Inductor_SMD:L_Chilisin_BWVS00505030, F.Cu at (95.1, 86.4)
- added NT1: NetTie_2, NetTie:NetTie-2_SMD_Pad0.5mm, F.Cu at (96.9, 78.6)
- added R26: 100k, Resistor_SMD:R_0402_1005Metric, F.Cu at (156.5, 99.0)
- added R27: 100k, Resistor_SMD:R_0402_1005Metric, F.Cu at (151.2, 97.0)
- added R28: 100k, Resistor_SMD:R_0402_1005Metric, F.Cu at (153.0, 97.0)
- added R29: 100k, Resistor_SMD:R_0402_1005Metric, F.Cu at (154.8, 97.0)
- added R30: 100k, Resistor_SMD:R_0402_1005Metric, F.Cu at (156.5, 97.0)
- added R31: 5.1k, Resistor_SMD:R_0402_1005Metric, F.Cu at (225.5, 113.8)
- added R36: 732k, Resistor_SMD:R_0402_1005Metric, F.Cu at (168.1, 87.9)
- added R6: 47Ω, Resistor_SMD:R_0402_1005Metric, F.Cu at (225.5, 109.8)
- added R7: 47Ω, Resistor_SMD:R_0402_1005Metric, F.Cu at (225.5, 111.8)
- added R9: 10mΩ, Resistor_SMD:R_1206_3216Metric, F.Cu at (98.5, 73.7)
- added TP1: TestPoint, TestPoint:TestPoint_Pad_D1.0mm, F.Cu at (182.8, 88.8)
- added TP3: TestPoint, TestPoint:TestPoint_Pad_D1.0mm, F.Cu at (182.8, 83.5)
- added TP4: TestPoint, TestPoint:TestPoint_Pad_D1.0mm, F.Cu at (182.8, 85.5)
- added U3: MAX17055ETB+T, YV:TDFN-10-EP-2x2p5-0p4mm, F.Cu at (93.7, 74.6)
- added U6: MT3608, Package_TO_SOT_SMD:SOT-23-6, F.Cu at (169.2, 82.7)
- C25: value 1nF -> 10uF
- J5: renamed from J9; footprint YV:ER-CON50HT-1 -> YV:HC-FPC-0.5-50P-FHH20
- R10, R8: value 5.1k -> 100k
- R11: value 180 -> 100k
- R12: value 10k -> 357Ω; footprint Resistor_SMD:R_0402_1005Metric -> Resistor_SMD:R_0603_1608Metric
- R16: value 10k -> 5.1k
- R21: value 10k -> 100k
- R22, R23: value 732k -> 100k
- R4: value 100 -> 100k
- R5: value 100 -> 31.6k
- moved R10 115.0 mm to (102.0, 84.2)
- moved R12 113.6 mm to (97.7, 76.6)
- moved R4 99.6 mm to (140.8, 97.9), turned to 0 degrees
- moved R8 96.2 mm to (168.8, 109.2)
- moved R16 92.7 mm to (219.2, 115.2)
- moved R21 82.9 mm to (151.2, 99.0), turned to -90 degrees
- moved R5 70.8 mm to (168.1, 85.9), turned to 0 degrees
- moved R11 39.7 mm to (102.0, 86.1), turned to 0 degrees
- moved R13 35.4 mm to (175.2, 81.2), turned to 0 degrees
- moved R22 20.5 mm to (153.0, 99.0), turned to -90 degrees
- moved R23 19.8 mm to (154.8, 99.0), turned to -90 degrees
- moved J3 18.0 mm to (156.8, 65.8), turned to -90 degrees
- moved C25 8.21 mm to (132.9, 90.2)
- moved D6 8.21 mm to (135.4, 85.4)
- moved Q2 8.21 mm to (134.7, 78.5)
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- renumbered C10 to C1, C9 to C14, C11 to C25, C8 to C26, C7 to C27, D2 to D6, D5 to D7, D4 to D8, J4 to J10, J5 to J11, J10 to J12, J3 to J13, J6 to J3, L4 to L8, Q1 to Q2, R9 to R32, R7 to R33, R6 to R34, R14 to R35, SW3 to SW1, SW1 to SW4, SW2 to SW5, U4 to U1, U3 to U4, U6 to U8
Connections:
- net /Power/Vin renamed /USB and Cells/Vin
- C25 pad 1: IO0(boot) -> Vbatt
- D7 pad 2: Net-(D4-A) -> Net-(D7-A)
- D8 pad 2: Net-(D4-A) -> Net-(D7-A)
- J1 pad 1: Vbatt -> Net-(J1-Pin_1)
- J10 pad A4: V-USB -> Net-(F3-Pad1)
- J10 pad A5: Net-(J4-CC1) -> Net-(J10-CC1)
- J10 pad A6: D+ -> Net-(J10-D+-PadA6)
- J10 pad A7: D- -> Net-(J10-D--PadA7)
- J10 pad A9: V-USB -> Net-(F3-Pad1)
- J10 pad B4: V-USB -> Net-(F3-Pad1)
- J10 pad B5: Net-(J4-CC2) -> Net-(J10-CC2)
- J10 pad B6: D+ -> Net-(J10-D+-PadA6)
- J10 pad B7: D- -> Net-(J10-D--PadA7)
- J10 pad B9: V-USB -> Net-(F3-Pad1)
- J11 pad 10: IO21 -> IO35
- J11 pad 11: I34 -> IO37
- J11 pad 12: Vbatt-VN -> IO58-UART0-TX
- J11 pad 13: I35 -> IO59-UART0-RX
- J11 pad 3: IO26 -> IO43
- J11 pad 4: IO25 -> IO44
- J11 pad 5: IO27 -> IO45
- J11 pad 6: IO0(boot) -> IO46
- J11 pad 7: IO32 -> IO47
- J11 pad 8: IO22 -> IO48
- J12 pad 1: unconnected-(J10-DAT2-Pad1) -> /ESP32-S31/DATA2
- J12 pad 2: unconnected-(J10-DAT3/CD-Pad2) -> /ESP32-S31/DATA3
- J12 pad 3: unconnected-(J10-CMD-Pad3) -> /ESP32-S31/CMD
- J12 pad 4: unconnected-(J10-VDD-Pad4) -> +3.3V
- J12 pad 5: unconnected-(J10-CLK-Pad5) -> /ESP32-S31/CLK
- J12 pad 6: unconnected-(J10-VSS-Pad6) -> GND
- J12 pad 7: unconnected-(J10-DAT0-Pad7) -> /ESP32-S31/DATA0
- J12 pad 8: unconnected-(J10-DAT1-Pad8) -> /ESP32-S31/DATA1
- J12 pad G1: unconnected-(J10-GND-PadG1) -> GND
- J12 pad G2: unconnected-(J10-GND-PadG2) -> GND
- J12 pad G3: unconnected-(J10-GND-PadG3) -> GND
- J12 pad G4: unconnected-(J10-GND-PadG4) -> GND
- J13 pad 3: IO14 -> IO57
- J13 pad 4: IO12 -> IO56
- J13 pad 5: IO13 -> IO55
- J13 pad 6: IO15 -> IO54
- J2 pad 1: Vbatt -> Net-(J2-Pin_1)
- J3 pad 1: unconnected-(J6-Pin_1-Pad1) -> /ESP32-S31/Touch-RST
- J3 pad 2: unconnected-(J6-Pin_2-Pad2) -> +3.3V
- J3 pad 3: unconnected-(J6-Pin_3-Pad3) -> GND
- J3 pad 4: unconnected-(J6-Pin_4-Pad4) -> /ESP32-S31/Touch-INT
- J3 pad 5: unconnected-(J6-Pin_5-Pad5) -> /ESP32-S31/I2C1-SDA
- J3 pad 6: unconnected-(J6-Pin_6-Pad6) -> /ESP32-S31/I2C1-SCL
- J5 pad 1: unconnected-(J9-Pin_1-Pad1) -> +3.3V
- J5 pad 10: unconnected-(J9-Pin_10-Pad10) -> /ESP32-S31/DS16
- J5 pad 11: unconnected-(J9-Pin_11-Pad11) -> GND
- J5 pad 12: unconnected-(J9-Pin_12-Pad12) -> /ESP32-S31/DS15
- J5 pad 13: unconnected-(J9-Pin_13-Pad13) -> /ESP32-S31/DS14
- J5 pad 14: unconnected-(J9-Pin_14-Pad14) -> /ESP32-S31/DS13
- J5 pad 15: unconnected-(J9-Pin_15-Pad15) -> /ESP32-S31/DS12
- J5 pad 16: unconnected-(J9-Pin_16-Pad16) -> /ESP32-S31/DS11
- J5 pad 17: unconnected-(J9-Pin_17-Pad17) -> /ESP32-S31/DS10
- J5 pad 18: unconnected-(J9-Pin_18-Pad18) -> /ESP32-S31/DS9
- J5 pad 19: unconnected-(J9-Pin_19-Pad19) -> /ESP32-S31/DS8
- J5 pad 2: unconnected-(J9-Pin_2-Pad2) -> +3.3V
- J5 pad 20: unconnected-(J9-Pin_20-Pad20) -> GND
- J5 pad 21: unconnected-(J9-Pin_21-Pad21) -> /ESP32-S31/DS7
- J5 pad 22: unconnected-(J9-Pin_22-Pad22) -> /ESP32-S31/DS6
- J5 pad 23: unconnected-(J9-Pin_23-Pad23) -> /ESP32-S31/DS5
- J5 pad 24: unconnected-(J9-Pin_24-Pad24) -> /ESP32-S31/DS4
- J5 pad 25: unconnected-(J9-Pin_25-Pad25) -> /ESP32-S31/DS3
- J5 pad 26: unconnected-(J9-Pin_26-Pad26) -> /ESP32-S31/DS2
- J5 pad 27: unconnected-(J9-Pin_27-Pad27) -> /ESP32-S31/DS1
- J5 pad 28: unconnected-(J9-Pin_28-Pad28) -> /ESP32-S31/DS0
- J5 pad 29: unconnected-(J9-Pin_29-Pad29) -> GND
- J5 pad 3: unconnected-(J9-Pin_3-Pad3) -> /ESP32-S31/DS23
- J5 pad 30: unconnected-(J9-Pin_30-Pad30) -> /ESP32-S31/PCLK
- J5 pad 31: unconnected-(J9-Pin_31-Pad31) -> /ESP32-S31/HS
- J5 pad 32: unconnected-(J9-Pin_32-Pad32) -> /ESP32-S31/VS
- J5 pad 33: unconnected-(J9-Pin_33-Pad33) -> /ESP32-S31/DE
- J5 pad 34: unconnected-(J9-Pin_34-Pad34) -> /ESP32-S31/SD0
- J5 pad 35: unconnected-(J9-Pin_35-Pad35) -> /ESP32-S31/CS
- J5 pad 36: unconnected-(J9-Pin_36-Pad36) -> GND
- J5 pad 37: unconnected-(J9-Pin_37-Pad37) -> /ESP32-S31/SCL
- J5 pad 39: unconnected-(J9-Pin_39-Pad39) -> /ESP32-S31/SDA
- J5 pad 4: unconnected-(J9-Pin_4-Pad4) -> /ESP32-S31/DS22
- J5 pad 40: unconnected-(J9-Pin_40-Pad40) -> /ESP32-S31/RST
- J5 pad 41: unconnected-(J9-Pin_41-Pad41) -> /Screen/TE
- J5 pad 43: unconnected-(J9-Pin_43-Pad43) -> +14.5V
- J5 pad 45: unconnected-(J9-Pin_45-Pad45) -> GND
- J5 pad 47: unconnected-(J9-Pin_47-Pad47) -> /Screen/IM3
- J5 pad 48: unconnected-(J9-Pin_48-Pad48) -> /Screen/IM2
- J5 pad 49: unconnected-(J9-Pin_49-Pad49) -> /Screen/IM1
- J5 pad 5: unconnected-(J9-Pin_5-Pad5) -> /ESP32-S31/DS21
- J5 pad 50: unconnected-(J9-Pin_50-Pad50) -> /Screen/IM0
- J5 pad 6: unconnected-(J9-Pin_6-Pad6) -> /ESP32-S31/DS20
- J5 pad 7: unconnected-(J9-Pin_7-Pad7) -> /ESP32-S31/DS19
- J5 pad 8: unconnected-(J9-Pin_8-Pad8) -> /ESP32-S31/DS18
- J5 pad 9: unconnected-(J9-Pin_9-Pad9) -> /ESP32-S31/DS17
- J7 pad 1: GND -> GNDREF
- J8 pad 1: GND -> GNDREF
- R10 pad 1: Net-(J4-CC1) -> +3.3V
- R10 pad 2: GND -> /ESP32-S31/I2C1-SCL
- R11 pad 1: Net-(D4-A) -> +3.3V
- R11 pad 2: V-USB -> /ESP32-S31/I2C1-SDA
- R12 pad 1: Net-(Q2-B) -> V-USB
- R12 pad 2: DTR -> Net-(D7-A)
- R13 pad 1: V-USB -> +3.3V
- R13 pad 2: GND -> /DC-DC/BACKLIGHTen
- R16 pad 1: Net-(Q3-B) -> Net-(J10-CC1)
- R16 pad 2: RTS -> GND
- R21 pad 1: +3.3V -> /Screen/IM3
- R21 pad 2: unconnected-(R21-Pad2) -> +3.3V
- R22 pad 1: Net-(JP1-A) -> /Screen/IM2
- R22 pad 2: Vbatt -> +3.3V
- R23 pad 1: GND -> /Screen/IM1
- R23 pad 2: Net-(JP1-A) -> +3.3V
- R4 pad 1: unconnected-(R4-Pad1) -> V-USB
- R4 pad 2: TXDtoRXD0 -> GND
- R5 pad 1: unconnected-(R5-Pad1) -> Net-(U6-FB)
- R5 pad 2: RXDtoTXD0 -> GND
- R8 pad 1: Net-(J4-CC2) -> +3.3V
- R8 pad 2: GND -> EN
- SW5 pad 1: IO0(boot) -> BOOT
- U1 pad 10: unconnected-(U4-GPIO4-Pad10) -> /ESP32-S31/DS0
- U1 pad 11: unconnected-(U4-GPIO5-Pad11) -> /ESP32-S31/DS1
- U1 pad 12: unconnected-(U4-GPIO6-Pad12) -> /ESP32-S31/DS2
- U1 pad 13: unconnected-(U4-GPIO7-Pad13) -> /ESP32-S31/DS3
- U1 pad 14: unconnected-(U4-GPIO8-Pad14) -> /ESP32-S31/DS4
- U1 pad 15: unconnected-(U4-GPIO9-Pad15) -> /ESP32-S31/DS8
- U1 pad 16: unconnected-(U4-GPIO10-Pad16) -> /ESP32-S31/DS9
- U1 pad 17: unconnected-(U4-GPIO11-Pad17) -> /ESP32-S31/DS10
- U1 pad 18: unconnected-(U4-GPIO12-Pad18) -> /ESP32-S31/DS11
- U1 pad 19: unconnected-(U4-GPIO13-Pad19) -> /ESP32-S31/DS12
- U1 pad 20: unconnected-(U4-GPIO14-Pad20) -> /ESP32-S31/DS13
- U1 pad 21: unconnected-(U4-GPIO15-Pad21) -> /ESP32-S31/DS16
- U1 pad 22: unconnected-(U4-GPIO16-Pad22) -> /ESP32-S31/DS17
- U1 pad 23: unconnected-(U4-GPIO17-Pad23) -> /ESP32-S31/DS18
- U1 pad 24: unconnected-(U4-GPIO18-Pad24) -> /ESP32-S31/DS19
- U1 pad 25: unconnected-(U4-GPIO19-Pad25) -> /ESP32-S31/DS20
- U1 pad 27: unconnected-(U4-SDIO_DATA0/GPIO20-Pad27) -> /ESP32-S31/DATA0
- U1 pad 28: unconnected-(U4-SDIO_DATA1/GPIO21-Pad28) -> /ESP32-S31/DATA1
- U1 pad 29: unconnected-(U4-SDIO_DATA2/GPIO22-Pad29) -> /ESP32-S31/DATA2
- U1 pad 3: unconnected-(U4-3V3-Pad3) -> +3.3V
- U1 pad 30: unconnected-(U4-SDIO_DATA3/GPIO23-Pad30) -> /ESP32-S31/DATA3
- U1 pad 31: unconnected-(U4-SDIO_CLK/GPIO24-Pad31) -> /ESP32-S31/CLK
- U1 pad 32: unconnected-(U4-SDIO_CMD/GPIO25-Pad32) -> /ESP32-S31/CMD
- U1 pad 4: unconnected-(U4-3V3-Pad4) -> +3.3V
- U1 pad 40: unconnected-(U4-USB_DP-Pad40) -> Net-(U1-USB_DP)
- U1 pad 41: unconnected-(U4-USB_DM-Pad41) -> Net-(U1-USB_DM)
- U1 pad 42: unconnected-(U4-GPIO33-Pad42) -> /ESP32-S31/USB-Dn
- U1 pad 43: unconnected-(U4-GPIO34-Pad43) -> /ESP32-S31/USB-Dp
- U1 pad 44: D+ -> IO35
- U1 pad 45: D- -> Net-(U1-GPIO36*)
- U1 pad 46: unconnected-(U4-GPIO37-Pad46) -> IO37
- U1 pad 49: unconnected-(U4-GPIO38-Pad49) -> /ESP32-S31/DE
- U1 pad 5: unconnected-(U4-EN-Pad5) -> EN
- U1 pad 50: unconnected-(U4-GPIO39-Pad50) -> /ESP32-S31/VS
- U1 pad 51: unconnected-(U4-GPIO40-Pad51) -> /ESP32-S31/HS
- U1 pad 52: unconnected-(U4-GPIO42/ADC1_CH0_N-Pad52) -> /ESP32-S31/PCLK
- U1 pad 53: unconnected-(U4-GPIO43/ADC1_CH0_P-Pad53) -> IO43
- U1 pad 54: unconnected-(U4-GPIO44/ADC1_CH1_N-Pad54) -> IO44
- U1 pad 55: unconnected-(U4-GPIO45/ADC1_CH1_P-Pad55) -> IO45
- U1 pad 56: unconnected-(U4-GPIO46/ADC1_CH2_N-Pad56) -> IO46
- U1 pad 57: unconnected-(U4-GPIO47/ADC1_CH2_P-Pad57) -> IO47
- U1 pad 58: unconnected-(U4-GPIO48/ADC1_CH3_N-Pad58) -> IO48
- U1 pad 59: unconnected-(U4-GPIO49/ADC1_CH3_P-Pad59) -> /ESP32-S31/RST
- U1 pad 6: unconnected-(U4-GPIO2-Pad6) -> /ESP32-S31/Touch-RST
- U1 pad 60: unconnected-(U4-GPIO50/ADC2_CH0_N-Pad60) -> /ESP32-S31/CS
- U1 pad 61: unconnected-(U4-GPIO51/ADC2_CH0_P-Pad61) -> /ESP32-S31/SDA
- U1 pad 62: unconnected-(U4-GPIO52/ADC2_CH1_N-Pad62) -> /ESP32-S31/SCL
- U1 pad 63: unconnected-(U4-GPIO53/ADC2_CH1_P-Pad63) -> /ESP32-S31/SD0
- U1 pad 64: unconnected-(U4-MTDO/GPIO54-Pad64) -> IO54
- U1 pad 65: unconnected-(U4-MTCK/GPIO55-Pad65) -> IO55
- U1 pad 66: unconnected-(U4-MTDI/GPIO56-Pad66) -> IO56
- U1 pad 67: unconnected-(U4-MTMS/GPIO57-Pad67) -> IO57
- U1 pad 68: unconnected-(U4-UART0_TXD/GPIO58-Pad68) -> IO58-UART0-TX
- U1 pad 69: unconnected-(U4-UART0_RXD/GPIO59-Pad69) -> IO59-UART0-RX
- U1 pad 7: unconnected-(U4-GPIO3-Pad7) -> /ESP32-S31/Touch-INT
- U1 pad 70: unconnected-(U4-GPIO60-Pad70) -> /DC-DC/BACKLIGHTen
- U1 pad 71: unconnected-(U4-GPIO61-Pad71) -> BOOT
- U1 pad 8: unconnected-(U4-GPIO0/XTAL_32K_N-Pad8) -> /ESP32-S31/I2C1-SDA
- U1 pad 9: unconnected-(U4-GPIO1/XTAL_32K_P-Pad9) -> /ESP32-S31/I2C1-SCL
Routing:
- net Batt-Monitor: track 46.5 -> 0.00 mm
- net (no net): track 17.7 -> 0.70 mm
- net Net-(JP1-A): track 17.0 -> 0.00 mm, vias 1 -> 0
- net IO15: track 11.7 -> 0.00 mm
- net IO25: track 9.31 -> 0.00 mm
- net Vbatt: track 51.6 -> 45.7 mm
- net Vbatt-VN: track 3.84 -> 0.00 mm
- net IO12: track 2.67 -> 0.00 mm
- net GND: track 53.0 -> 51.2 mm, vias 44 -> 42
- net V-USB: track 14.0 -> 13.5 mm
- net /USB and Cells/Vin: vias 15 -> 13
- net /ESP32-S31/DS15: vias 0 -> 1
- net /ESP32-S31/DS13: vias 0 -> 1
- net +5V: vias 12 -> 13

Commit message: Flip the connector and Pot in the layout
Other:
- outline, holes or cut-outs redrawn
Changed lines of the file:
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@@
 		(layer "B.SilkS")
 	)
-	(gr_line
-		(start 111.75 117.002)
-		(end 111.75 50.8)
-		(stroke
-			(width 0.15)
-			(type default)
-		)
-		(layer "Edge.Cuts")
-	)
 	(gr_arc
-		(start 111.750637 50.793108)
-		(mid 111.984952 50.227423)
-		(end 112.550637 49.993108)
+		(start 111.75 51)
+		(mid 112.042893 50.292893)
+		(end 112.75 50)
 		(stroke
 			(width 0.15)
@@
 	)
 	(gr_line
-		(start 112.550637 50)
-		(end 214.4 50)
+		(start 111.75 116.202)
+		(end 111.75 51)
 		(stroke
 			(width 0.15)
@@
 		(stroke
 			(width 0.15)
+			(type default)
+		)
+		(layer "Edge.Cuts")
+	)
+	(gr_line
+		(start 112.75 50)
+		(end 214.4 50)
+		(stroke
+			(width 0.15)
