File: Hardware/esp32-V2.kicad_pcb (KiCad board)
At the start: 4 copper layers, 103.7 x 68 mm, 120 parts, among them J1 Conn_01x01_Socket, J10 HC-FPC-0.5-50P-FHH20, J2 Conn_01x01_Socket, J3 Conn_01x08_F_Header, J4 MSD-4-A, J5 PM254-1-17-Z-8.5, J6 USB_C_Receptacle-16p, J7 Conn_01x01_Socket, J8 Conn_01x01_Socket, J9 KH-FG0.5-H2.0-6PIN, Q1 DMP3015LSS-13, SW1 SW_Push_DPDT, SW2 SW-000001, SW3 SW-000001, U1 TPS61170DRVR, U2 IC-TPS61022, U3 ESP32-S31-WROOM-3-N16R16V, U4 LT1963AEST-3.3#TRPBF, U5 CN3158, U6 TPS63700, U7 MT3608, U8 MAX17055ETB+T

Commit message: Gerbers Generation
Parts:
- removed C22: 10uF, Capacitor_SMD:C_0402_1005Metric
- moved REF** 2.55 mm to (135.5, 70.5)
