File: Hardware/power.kicad_sch (KiCad schematic)
At the start: 61 parts, among them J1 Conn_01x01_Socket, J2 Conn_01x01_Socket, J4 USB_C_Receptacle_USB2.0_16P, J7 Conn_01x01_Socket, J8 Conn_01x01_Socket, Q1 DMP3015LSS-13, SW3 SW_Push_DPDT, U2 TPS61170DRVR, U3 TPS61022, U5 LT1963AEST-3.3#TRPBF, U6 CN3158, U7 TPS63700

Commit message: New BaseBoard
Parts:
- removed C10, C11: 10uF, Capacitor_SMD:C_0402_1005Metric, symbol Device:C
- removed C7, C8, C9: 22uF, Capacitor_SMD:C_0805_2012Metric, symbol Device:C
- removed D2: Fuxinsemi_PDS760, Package_TO_SOT_SMD:TO-277B, symbol Diode:Fuxinsemi_PDS760
- removed D4: Green, 3.2V, LED_SMD:LED_0603_1608Metric, symbol LED:CQY99
- removed D5: Blue 2.9V, LED_SMD:LED_0603_1608Metric, symbol LED:CQY99
- removed J1, J2, J7, J8: Conn_01x01_Socket, Battery:BatteryClip_Keystone_54_D16-19mm, symbol Connector:Conn_01x01_Socket
- removed J4: USB_C_Receptacle_USB2.0_16P, Connector_USB:USB_C_Receptacle_GCT_USB4105-xx-A_16P_TopMnt_Horizontal, symbol Connector:USB_C_Receptacle_USB2.0_16P
- removed L4: 1uH, Inductor_SMD:L_Coilcraft_XAL5030-XXX, symbol Device:L
- removed Q1: DMP3015LSS-13, Package_SO:SOIC-8_3.9x4.9mm_P1.27mm, symbol Transistor_FET:IRF7606PBF
- removed R10, R8: 5.1k, Resistor_SMD:R_0402_1005Metric, symbol Device:R
- removed R11: 180, Resistor_SMD:R_0402_1005Metric, symbol Device:R
- removed R13, R6, R9: 100k, Resistor_SMD:R_0402_1005Metric, symbol Device:R
- removed R14: 1.18k, Resistor_SMD:R_0402_1005Metric, symbol Device:R
- removed R7: 732k, Resistor_SMD:R_0402_1005Metric, symbol Device:R
- removed SW3: SW_Push_DPDT, Button_Switch_THT:SW_CK_JS202011AQN_DPDT_Angled, symbol Switch:SW_Push_DPDT
- removed U3: TPS61022, Package_DFN_QFN:Texas_RWU0007A_VQFN-7_2x2mm_P0.5mm, symbol Converter_DCDC:TPS61022
- removed U6: CN3158, YV:SOIC-8-1EP_3.9x4.9mm_P1.27mm_EP2.41x3.3mm_ThermalVias-0p3mm, symbol Battery_Management:CN3158
Connections:
- no-connect marks 6 -> 0
Other:
- note added: "15V"
- note removed: "2x18650 cell 3.2V LiFePO4"
- note removed: "BATT / USB TO 5V"
- note removed: "LiFePO4 BATTERIES"
- note removed: "LiFePO4 BATTERIES CHARGER"
- note removed: "USB C"
- note removed: "battery charger"
- note removed: "cell to 5V"
- note removed: "pwm mode"

Commit message: Schematic Done
Parts:
- removed L2, L7: 10uH, Inductor_SMD:L_Chilisin_BWVS00505030, symbol Device:L
- added C30, C33, C34, C35: 4.7uF, Capacitor_SMD:C_0402_1005Metric, symbol Device:C
- added C9: 10uF, Capacitor_SMD:C_0402_1005Metric, symbol Device:C
- added D15: D_Schottky, Diode_SMD:D_SOD-123F, symbol Device:D_Schottky
- added L2, L7, L9: 10uH, Inductor_SMD:L_Chilisin_BWVS00505030, symbol YV-library:IND10U0Z1A20-00
- added R36: 732k, Resistor_SMD:R_0402_1005Metric, symbol Device:R
- added R5: 31.6k, Resistor_SMD:R_0402_1005Metric, symbol YV-library:RES31K6M-00
- added U6: MT3608, Package_TO_SOT_SMD:SOT-23-6, symbol YV-library:MT3608
Connections:
- net +5V: now also C9.1, L9.1, U6.5 (IN)
- net GND: now also C30.2, C33.2, C34.2, C35.2, C9.2, L7.1, R5.2, U6.2 (GND)
- net at D3.1 (K), U7.6 (SW): now also L7.2
- net at C6.1, L3.2, U2.5 (CTRL)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: now also L2.1
- net at D1.2 (A), U2.4 (SW): now also L2.2
- new net: D15.2 (A), L9.2, U6.1 (SW)
- new net: R36.1, R5.1, U6.3 (FB)
- new net +14.5V: C30.1, C33.1, C34.1, C35.1, D15.1 (K), R36.2
- new net BACKLIGHTen: U6.4 (EN)
Other:
- note added: "+5V TO +14.5V LCD's BackLight"
- note added: "1.2 MHz"
- note added: "30mA max"
- note removed: "15V"
- company: (none) -> Motion Composites
- title: (none) -> Strain Gauge Data Logger
- moved on the sheet: C12, C13, D1, U5

Commit message: Layout cleaned
Parts:
- renumbered C12 to C14, C30 to C18, C33 to C19, C35 to C20, C34 to C21, C18 to C23, C19 to C24, C20 to C25, C21 to C26, C22 to C27, C23 to C28, C9 to C29, C24 to C30, C6 to C7, D3 to D10, D15 to D11, D1 to D7, L9 to L8, R17 to R12, R18 to R13, R19 to R15, R36 to R16, R5 to R17, R20 to R18, R1 to R2, R2 to R4, R3 to R6, U2 to U1, U5 to U4, U7 to U6, U6 to U7

Commit message: Update de la librairy et du BOM
Parts:
- C13, C14, C28, C29, C7: symbol Device:C -> YV-library:CAPX10U0M6V30-00; LCSC C20069813 -> C15525; PartNumber CSA0402X7R474K100GT -> CL05A106MQ5NUNC
- C15, C23: symbol Device:C -> YV-library:CAPX220NM25V0-00
- C16: symbol Device:C -> YV-library:CAPN10P0M50V0-00
- C17, C4, C5: symbol Device:C -> YV-library:CAPN4N70M50V0-00
- C18, C19, C20, C21, C24, C25, C26, C27, C3: symbol Device:C -> YV-library:CAPX4U70M25V0-00
- C2, C30: symbol Device:C_Polarized_US -> YV-library:CAPA20U0Z35V0-00
- D10, D11, D7: value D_Schottky -> Diode-DK24; symbol Device:D_Schottky -> YV-library:Diode-DK24
- L1, L3, L5, L6: symbol Device:L_Ferrite -> YV-library:Ferrite-BWVS00505030
- R12: symbol Device:R -> YV-library:RES150KM-00
- R13: symbol Device:R -> YV-library:RES100KM-00; LCSC C2909355 -> C25741; PartNumber (none) -> 0402WGF1003TCE
- R15: symbol Device:R -> YV-library:RES1M54M-00
- R16: symbol Device:R -> YV-library:RES732KM-00; PartNumber (none) -> 0402WGF7323TCE
- R18: symbol Device:R -> YV-library:RES10R0M-00
- R2: symbol Device:R -> YV-library:RES10K0M-00; PartNumber (none) -> 0402WGF1002TCE
- R4: symbol Device:R -> YV-library:RES91K0M-00
- R6: symbol Device:R -> YV-library:RES10K0M-00
- U1: PartNumber (none) -> TPS61170DRVR
- U4: symbol Regulator_Linear:LT1963AxST-1.5 -> YV-library:IC-LT1963AEST-3.3
